File: hardware/pcb/stm32_car_drive_v2.0.0/bb68942b.kicad_sch (KiCad schematic)
At the start: 12 parts, among them J2 Conn_01x06, J4 Conn_01x06, U5 DRV8870DDA, U8 DRV8870DDA

Commit message: update
Changed lines of the file:
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@@
 		)
 	)
-	(label "AENO1"
-		(at 231.14 71.12 180)
+	(label "BOUT2"
+		(at 154.94 129.54 0)
 		(fields_autoplaced yes)
 		(effects
@@
 				(size 1.27 1.27)
 			)
-			(justify right bottom)
-		)
-	)
-	(label "BOUT2"
-		(at 154.94 129.54 0)
+			(justify left bottom)
+		)
+	)
+	(label "BOUT1"
+		(at 154.94 127 0)
 		(fields_autoplaced yes)
 		(effects
@@
 		)
 	)
-	(label "BENO2"
-		(at 231.14 97.79 180)
+	(label "AOUT1"
+		(at 231.14 78.74 180)
 		(fields_autoplaced yes)
 		(effects
@@
 		)
 	)
-	(label "DIRA"
-		(at 59.69 93.98 0)
+	(label "AOUT2"
+		(at 231.14 66.04 180)
 		(fields_autoplaced yes)
 		(effects
@@
 				(size 1.27 1.27)
 			)
-			(justify left bottom)
-		)
-	)
-	(label "BENO1"
-		(at 231.14 95.25 180)
+			(justify right bottom)
+		)
+	)
+	(label "AOUT1"
+		(at 156.21 39.37 0)
 		(fields_autoplaced yes)
 		(effects
@@
 				(size 1.27 1.27)
 			)
-			(justify right bottom)
-		)
-	)
-	(label "PWMB"
-		(at 60.96 127 0)
+			(justify left bottom)
+		)
+	)
+	(label "AOUT2"
+		(at 156.21 41.91 0)
 		(fields_autoplaced yes)
 		(effects
@@
 		)
 	)
-	(label "AENO2"
-		(at 231.14 73.66 180)
+	(label "BOUT1"
+		(at 231.14 102.87 180)
 		(fields_autoplaced yes)
 		(effects
@@
 		)
 	)
-	(label "DIRB"
-		(at 60.96 140.97 0)
+	(hierarchical_label "PWMB"
+		(shape input)
+		(at 60.96 175.26 180)
 		(fields_autoplaced yes)
 		(effects
@@
 				(size 1.27 1.27)
 			)
-			(justify left bottom)
-		)
-	)
-	(label "BOUT1"
-		(at 154.94 127 0)
+			(justify right)
+		)
+	)
+	(hierarchical_label "DIRB"
+		(shape input)
+		(at 60.96 181.61 180)
 		(fields_autoplaced yes)
 		(effects
@@
 				(size 1.27 1.27)
 			)
-			(justify left bottom)
-		)
-	)
-	(label "AOUT1"
-		(at 231.14 78.74 180)
+			(justify right)
+		)
+	)
+	(hierarchical_label "DIRA"
+		(shape input)
+		(at 59.69 53.34 180)
 		(fields_autoplaced yes)
 		(effects
@@
 				(size 1.27 1.27)
 			)
-			(justify right bottom)
-		)
-	)
-	(label "DIRA"
-		(at 59.69 53.34 0)
+			(justify right)
+		)
+	)
+	(hierarchical_label "PWMA"
+		(shape input)
+		(at 59.69 87.63 180)
 		(fields_autoplaced yes)
 		(effects
@@
 				(size 1.27 1.27)
 			)
-			(justify left bottom)
-		)
-	)
-	(label "PWMA"
-		(at 59.69 39.37 0)
+			(justify right)
+		)
+	)
+	(hierarchical_label "DIRB"
+		(shape input)
+		(at 60.96 140.97 180)
 		(fields_autoplaced yes)
 		(effects
@@
 				(size 1.27 1.27)
 			)
-			(justify left bottom)
-		)
-	)
-	(label "AOUT2"
-		(at 231.14 66.04 180)
+			(justify right)
+		)
+	)
+	(hierarchical_label "AENO1"
+		(shape input)
+		(at 231.14 71.12 0)
 		(fields_autoplaced yes)
 		(effects
@@
 				(size 1.27 1.27)
 			)
-			(justify right bottom)
-		)
-	)
-	(label "PWMB"
-		(at 60.96 175.26 0)
+			(justify left)
+		)
+	)
+	(hierarchical_label "PWMB"
+		(shape input)
+		(at 60.96 127 180)
 		(fields_autoplaced yes)
 		(effects
@@
 				(size 1.27 1.27)
 			)
-			(justify left bottom)
-		)
-	)
-	(label "AOUT1"
-		(at 156.21 39.37 0)
+			(justify right)
+		)
+	)
+	(hierarchical_label "AENO2"
+		(shape input)
+		(at 231.14 73.66 0)
 		(fields_autoplaced yes)
 		(effects
@@
 				(size 1.27 1.27)
 			)
-			(justify left bottom)
-		)
-	)
-	(label "AOUT2"
-		(at 156.21 41.91 0)
+			(justify left)
+		)
+	)
+	(hierarchical_label "BENO2"
+		(shape input)
+		(at 231.14 97.79 0)
 		(fields_autoplaced yes)
 		(effects
@@
 				(size 1.27 1.27)
 			)
-			(justify left bottom)
-		)
-	)
-	(label "PWMA"
-		(at 59.69 87.63 0)
+			(justify left)
+		)
+	)
+	(hierarchical_label "BENO1"
+		(shape input)
+		(at 231.14 95.25 0)
 		(fields_autoplaced yes)
 		(effects
@@
 				(size 1.27 1.27)
 			)
-			(justify left bottom)
-		)
-	)
-	(label "BOUT1"
-		(at 231.14 102.87 180)
+			(justify left)
+		)
+	)
+	(hierarchical_label "DIRA"
+		(shape input)
+		(at 59.69 93.98 180)
 		(fields_autoplaced yes)
 		(effects
@@
 				(size 1.27 1.27)
 			)
-			(justify right bottom)
-		)
-	)
-	(label "DIRB"
-		(at 60.96 181.61 0)
+			(justify right)
+		)
+	)
+	(hierarchical_label "PWMA"
+		(shape input)
+		(at 59.69 39.37 180)
 		(fields_autoplaced yes)
 		(effects
@@
 				(size 1.27 1.27)
 			)
-			(justify left bottom)
-		)
-	)
-	(hierarchical_label "PWMB"
-		(shape input)
-		(at 60.96 175.26 180)
-		(fields_autoplaced yes)
-		(effects
-			(font
-				(size 1.27 1.27)
-			)
-			(justify right)
-		)
-	)
-	(hierarchical_label "DIRB"
-		(shape input)
-		(at 60.96 181.61 180)
-		(fields_autoplaced yes)
-		(effects
-			(font
-				(size 1.27 1.27)
-			)
-			(justify right)
-		)
-	)
-	(hierarchical_label "DIRA"
-		(shape input)
-		(at 59.69 53.34 180)
-		(fields_autoplaced yes)
-		(effects
-			(font
-				(size 1.27 1.27)
-			)
-			(justify right)
-		)
-	)
-	(hierarchical_label "PWMA"
-		(shape input)
-		(at 59.69 87.63 180)
-		(fields_autoplaced yes)
-		(effects
-			(font
-				(size 1.27 1.27)
-			)
-			(justify right)
-		)
-	)
-	(hierarchical_label "DIRB"
-		(shape input)
-		(at 60.96 140.97 180)
-		(fields_autoplaced yes)
-		(effects
-			(font
-				(size 1.27 1.27)
-			)
-			(justify right)
-		)
-	)
-	(hierarchical_label "AENO1"
-		(shape input)
-		(at 231.14 71.12 0)
-		(fields_autoplaced yes)
-		(effects
-			(font
-				(size 1.27 1.27)
-			)
-			(justify left)
-		)
-	)
-	(hierarchical_label "PWMB"
-		(shape input)
-		(at 60.96 127 180)
-		(fields_autoplaced yes)
-		(effects
-			(font
-				(size 1.27 1.27)
-			)
-			(justify right)
-		)
-	)
-	(hierarchical_label "AENO2"
-		(shape input)
-		(at 231.14 73.66 0)
-		(fields_autoplaced yes)
-		(effects
-			(font
-				(size 1.27 1.27)
-			)
-			(justify left)
-		)
-	)
-	(hierarchical_label "BENO2"
-		(shape input)
-		(at 231.14 97.79 0)
-		(fields_autoplaced yes)
-		(effects
-			(font
-				(size 1.27 1.27)
-			)
-			(justify left)
-		)
-	)
-	(hierarchical_label "BENO1"
-		(shape input)
-		(at 231.14 95.25 0)
-		(fields_autoplaced yes)
-		(effects
-			(font
-				(size 1.27 1.27)
-			)
-			(justify left)
-		)
-	)
-	(hierarchical_label "DIRA"
-		(shape input)
-		(at 59.69 93.98 180)
-		(fields_autoplaced yes)
-		(effects
-			(font
-				(size 1.27 1.27)
-			)
-			(justify right)
-		)
-	)
-	(hierarchical_label "PWMA"
-		(shape input)
-		(at 59.69 39.37 180)
-		(fields_autoplaced yes)
-		(effects
-			(font
-				(size 1.27 1.27)
-			)
 			(justify right)
 		)
@@
 	)
 	(symbol
-		(lib_name "CH443K_1")
 		(lib_id "Library:CH443K_1")
 		(at 86.36 31.75 0)
@@
 	)
 	(symbol
-		(lib_name "CH443K_3")
 		(lib_id "Library:CH443K_3")
 		(at 88.9 119.38 0)
@@
 	)
 	(symbol
-		(lib_name "CH443K_2")
 		(lib_id "Library:CH443K_2")
 		(at 87.63 72.39 0)
